File: schematics/schema3/schema3.sch (KiCad schematic (older format))
At the start: 11 parts, among them P1 LT293D, U1 LT1129CQ-3.3, U2 ESP-07, U3 7805

Commit message: Schematics
Parts:
- removed L1: VALVE, ~, symbol INDUCTOR
- removed R3: 7K, ~, symbol R
- removed R4: 1K, ~, symbol R
- added P2: CONN_2, symbol CONN_2
- added P3: USB-A-PCB, symbol USB-A-PCB
- renumbered BT to BT1, JP to JP1
Connections:
- net labels added: D+, D-
- wire segments 53 -> 60
- no-connect marks 0 -> 14
Other:
- moved on the sheet: JP1
Changed lines of the file:
@@
 LIBS:valves
 LIBS:ESP8266
+LIBS:ftdi
+LIBS:usb-b
+LIBS:ft232bm
+LIBS:USB
+LIBS:schema1 -cache
 EELAYER 27 0
 EELAYER END
@@
 Sheet 1 1
 Title ""
-Date "19 jun 2015"
+Date "20 jun 2015"
 Rev ""
 Comp ""
@@
 $EndComp
 $Comp
-L INDUCTOR L1
-U 1 1 5581C42C
-P 7950 1050
-F 0 "L1" V 7900 1050 40  0000 C CNN
-F 1 "VALVE" V 8050 1050 40  0000 C CNN
-F 2 "~" H 7950 1050 60  0000 C CNN
-F 3 "~" H 7950 1050 60  0000 C CNN
-	1    7950 1050
-	0    -1   -1   0
-$EndComp
-$Comp
 L ESP-07V2 U2
 U 1 1 5582A81F
@@
 $EndComp
 $Comp
-L BATTERY BT
+L BATTERY BT1
 U 1 1 5582A9C5
 P 3550 1600
-F 0 "BT" H 3550 1800 50  0000 C CNN
+F 0 "BT1" H 3550 1800 50  0000 C CNN
 F 1 "8V" H 3550 1410 50  0000 C CNN
 F 2 "~" H 3550 1600 60  0000 C CNN
@@
 $EndComp
 $Comp
-L GND #PWR?
+L GND #PWR01
 U 1 1 5582AA7E
 P 5650 4300
-F 0 "#PWR?" H 5650 4300 30  0001 C CNN
+F 0 "#PWR01" H 5650 4300 30  0001 C CNN
 F 1 "GND" H 5650 4230 30  0001 C CNN
 F 2 "" H 5650 4300 60  0000 C CNN
@@
 $EndComp
 $Comp
-L GND #PWR?
+L GND #PWR02
 U 1 1 5582AAF5
 P 5650 4300
-F 0 "#PWR?" H 5650 4300 30  0001 C CNN
+F 0 "#PWR02" H 5650 4300 30  0001 C CNN
 F 1 "GND" H 5650 4230 30  0001 C CNN
 F 2 "" H 5650 4300 60  0000 C CNN
@@
 $EndComp
 $Comp
-L GND #PWR?
-U 1 1 5582AC2C
-P 5000 100
-F 0 "#PWR?" H 5000 100 30  0001 C CNN
-F 1 "GND" H 5000 30  30  0001 C CNN
-F 2 "" H 5000 100 60  0000 C CNN
-F 3 "" H 5000 100 60  0000 C CNN
-	1    5000 100
-	1    0    0    -1
-$EndComp
-$Comp
-L GND #PWR?
-U 1 1 5582AC3B
-P 5100 1650
-F 0 "#PWR?" H 5100 1650 30  0001 C CNN
-F 1 "GND" H 5100 1580 30  0001 C CNN
-F 2 "" H 5100 1650 60  0000 C CNN
-F 3 "" H 5100 1650 60  0000 C CNN
-	1    5100 1650
-	1    0    0    -1
-$EndComp
-$Comp
-L GND #PWR?
-U 1 1 5582C77E
-P 6550 4300
-F 0 "#PWR?" H 6550 4300 30  0001 C CNN
-F 1 "GND" H 6550 4230 30  0001 C CNN
-F 2 "" H 6550 4300 60  0000 C CNN
-F 3 "" H 6550 4300 60  0000 C CNN
-	1    6550 4300
-	1    0    0    -1
-$EndComp
-$Comp
-L JUMPER JP
+L JUMPER JP1
 U 1 1 5582C7B4
-P 6800 3900
-F 0 "JP" H 6800 4050 60  0000 C CNN
-F 1 "JUMPER" H 6800 3820 40  0000 C CNN
-F 2 "~" H 6800 3900 60  0000 C CNN
-F 3 "~" H 6800 3900 60  0000 C CNN
-	1    6800 3900
+P 6800 3450
+F 0 "JP1" H 6800 3600 60  0000 C CNN
+F 1 "JUMPER" H 6800 3370 40  0000 C CNN
+F 2 "~" H 6800 3450 60  0000 C CNN
+F 3 "~" H 6800 3450 60  0000 C CNN
+	1    6800 3450
 	0    -1   -1   0
-$EndComp
-$Comp
-L GND #PWR?
-U 1 1 5582C7DC
-P 6800 4300
-F 0 "#PWR?" H 6800 4300 30  0001 C CNN
-F 1 "GND" H 6800 4230 30  0001 C CNN
-F 2 "" H 6800 4300 60  0000 C CNN
-F 3 "" H 6800 4300 60  0000 C CNN
-	1    6800 4300
-	1    0    0    -1
-$EndComp
-$Comp
-L GND #PWR?
-U 1 1 5582C80B
-P 7050 2050
-F 0 "#PWR?" H 7050 2050 30  0001 C CNN
-F 1 "GND" H 7050 1980 30  0001 C CNN
-F 2 "" H 7050 2050 60  0000 C CNN
-F 3 "" H 7050 2050 60  0000 C CNN
-	1    7050 2050
-	1    0    0    -1
 $EndComp
 $Comp
@@
 	1    0    0    -1
 $EndComp
-$Comp
-L GND #PWR?
-U 1 1 5582F347
-P 7500 4300
-F 0 "#PWR?" H 7500 4300 30  0001 C CNN
-F 1 "GND" H 7500 4230 30  0001 C CNN
-F 2 "" H 7500 4300 60  0000 C CNN
-F 3 "" H 7500 4300 60  0000 C CNN
-	1    7500 4300
-	1    0    0    -1
-$EndComp
+NoConn ~ 9350 2750
+NoConn ~ 9350 2850
+NoConn ~ 9350 2950
+NoConn ~ 9350 3050
+NoConn ~ 9350 3150
+NoConn ~ 9350 3250
+NoConn ~ 9350 3350
+NoConn ~ 4750 2700
+NoConn ~ 4750 2900
+NoConn ~ 4750 3000
+NoConn ~ 4750 3100
+NoConn ~ 4750 3200
+NoConn ~ 4650 1150
+$Comp
+L PWR_FLAG #FLG03
+U 1 1 5583E367
+P 4650 1000
+F 0 "#FLG03" H 4650 1095 30  0001 C CNN
+F 1 "PWR_FLAG" H 4650 1180 30  0000 C CNN
+F 2 "" H 4650 1000 60  0000 C CNN
+F 3 "" H 4650 1000 60  0000 C CNN
+	1    4650 1000
+	1    0    0    -1
+$EndComp
+$Comp
+L PWR_FLAG #FLG04
+U 1 1 5583EFE8
+P 5650 3800
+F 0 "#FLG04" H 5650 3895 30  0001 C CNN
+F 1 "PWR_FLAG" H 5650 3980 30  0000 C CNN
+F 2 "" H 5650 3800 60  0000 C CNN
+F 3 "" H 5650 3800 60  0000 C CNN
+	1    5650 3800
+	-1   0    0    1
+$EndComp
+$Comp
+L CONN_2 P2
+U 1 1 5584D826
+P 7950 700
+F 0 "P2" V 7900 700 40  0000 C CNN
+F 1 "CONN_2" V 8000 700 40  0000 C CNN
+F 2 "" H 7950 700 60  0000 C CNN
+F 3 "" H 7950 700 60  0000 C CNN
+	1    7950 700
+	0    -1   -1   0
+$EndComp
+$Comp
+L USB-A-PCB P3
+U 1 1 5584DD93
+P 2350 1200
+F 0 "P3" H 2350 1650 60  0000 C CNN
+F 1 "USB-A-PCB" H 2450 700 60  0000 C CNN
+F 2 "" H 2350 1200 60  0000 C CNN
+F 3 "" H 2350 1200 60  0000 C CNN
+	1    2350 1200
+	0    -1   -1   0
+$EndComp
+Text Label 2400 950  1    60   ~ 0
+D+
+Text Label 7900 5600 0    60   ~ 0
+D-
 Wire Wire Line
 	4750 2800 4200 2800
 Wire Wire Line
 	4200 2800 4200 2550
-Wire Wire Line
-	4200 1000 4200 2050
 Wire Wire Line
 	4750 2600 4600 2600
@@
 	3250 1600 3250 3800
 Wire Wire Line
-	3250 3800 5650 3800
+	3250 3800 7500 3800
 Wire Wire Line
 	5650 3800 5650 4300
@@
 	3850 1600 6650 1600
 Wire Wire Line
-	4200 1000 4650 1000
-Wire Wire Line
 	5550 1000 5650 1000
 Wire Wire Line
-	5100 1350 5100 1650
-Wire Wire Line
 	5550 1150 5550 1000
 Wire Wire Line
-	5650 1000 5650 2000
-Wire Wire Line
-	6550 3200 6550 4300
-Wire Wire Line
 	6550 3000 6800 3000
-Wire Wire Line
-	6800 3000 6800 3600
-Wire Wire Line
-	6800 4200 6800 4300
-Wire Wire Line
-	7050 1900 7050 2050
 Wire Wire Line
 	7450 1600 7450 2200
@@
 	8550 2950 7500 2950
 Wire Wire Line
-	7500 2950 7500 4300
-Wire Wire Line
 	6550 2900 7300 2900
 Wire Wire Line
@@
 	7300 3250 8550 3250
 Wire Wire Line
-	3850 1600 3850 1800
-$Comp
-L R R3
-U 1 1 5583BC3C
-P 3850 2050
-F 0 "R3" V 3930 2050 40  0000 C CNN
-F 1 "7K" V 3857 2051 40  0000 C CNN
-F 2 "~" V 3780 2050 30  0000 C CNN
-F 3 "~" H 3850 2050 30  0000 C CNN
-	1    3850 2050
-	1    0    0    -1
-$EndComp
-Wire Wire Line
-	3850 2300 3850 2800
-$Comp
-L R R4
-U 1 1 5583BC81
-P 3850 3050
-F 0 "R4" V 3930 3050 40  0000 C CNN
-F 1 "1K" V 3857 3051 40  0000 C CNN
-F 2 "~" V 3780 3050 30  0000 C CNN
-F 3 "~" H 3850 3050 30  0000 C CNN
-	1    3850 3050
-	1    0    0    -1
-$EndComp
-Wire Wire Line
-	3850 3300 3850 4300
-$Comp
-L GND #PWR?
-U 1 1 5583BCC7
-P 3850 4300
-F 0 "#PWR?" H 3850 4300 30  0001 C CNN
-F 1 "GND" H 3850 4230 30  0001 C CNN
-F 2 "" H 3850 4300 60  0000 C CNN
-F 3 "" H 3850 4300 60  0000 C CNN
-	1    3850 4300
-	1    0    0    -1
-$EndComp
-Wire Wire Line
-	3850 2700 4750 2700
-Connection ~ 3850 2700
+	4200 1000 4200 2050
+Wire Wire Line
+	4200 1000 4650 1000
+Connection ~ 3250 1950
+Wire Wire Line
+	6550 3800 6550 3200
+Connection ~ 5650 3800
+Wire Wire Line
+	6800 3800 6800 3750
+Connection ~ 6550 3800
+Wire Wire Line
+	6800 3000 6800 3150
+Wire Wire Line
+	7500 2950 7500 3800
+Connection ~ 6800 3800
+Wire Wire Line
+	7050 1900 7050 3800
+Connection ~ 7050 3800
+Wire Wire Line
+	3250 1950 5100 1950
+Wire Wire Line
+	5100 1950 5100 1350
+Wire Wire Line
+	7650 1050 7850 1050
+Wire Wire Line
+	8250 1050 8050 1050
+Wire Wire Line
+	2650 1600 3250 1600
+Connection ~ 5650 1000
+Wire Wire Line
+	2450 1600 2450 1850
+Wire Wire Line
+	2450 1850 6550 1850
+Wire Wire Line
+	6550 1850 6550 2600
+Wire Wire Line
+	2250 1600 2250 2100
+Wire Wire Line
+	2250 2100 6750 2100
+Wire Wire Line
+	6750 2100 6750 2700
+Wire Wire Line
+	6750 2700 6550 2700
+Wire Wire Line
+	5650 1000 5650 2000
+NoConn ~ 2050 1600
+$Comp
+L PWR_FLAG #FLG05
+U 1 1 5584E277
+P 6550 2700
+F 0 "#FLG05" H 6550 2795 30  0001 C CNN
+F 1 "PWR_FLAG" H 6550 2880 30  0000 C CNN
+F 2 "" H 6550 2700 60  0000 C CNN
+F 3 "" H 6550 2700 60  0000 C CNN
+	1    6550 2700
+	0    1    1    0
+$EndComp
 $EndSCHEMATC
