File: schematics/schema3/schema3 .sch (KiCad schematic (older format))
At the start: 10 parts, among them P1 LT293D, P2 CONN_2, P3 USB-A-PCB, U1 LT1129CQ-3.3, U2 ESP-07, U3 7805

Commit message: schematics changed
Parts:
- added R4: 7K, ~, symbol R
- added R5: 1K, ~, symbol R
Connections:
- wire segments 60 -> 64
- no-connect marks 14 -> 13
Changed lines of the file:
@@
 NoConn ~ 9350 3250
 NoConn ~ 9350 3350
-NoConn ~ 4750 2700
 NoConn ~ 4750 2900
 NoConn ~ 4750 3000
@@
 	0    1    1    0
 $EndComp
+Wire Wire Line
+	3900 1600 3900 2200
+Connection ~ 3900 1600
+$Comp
+L R R4
+U 1 1 55853C9B
+P 3900 2450
+F 0 "R4" V 3980 2450 40  0000 C CNN
+F 1 "7K" V 3907 2451 40  0000 C CNN
+F 2 "~" V 3830 2450 30  0000 C CNN
+F 3 "~" H 3900 2450 30  0000 C CNN
+	1    3900 2450
+	1    0    0    -1
+$EndComp
+Wire Wire Line
+	3900 2700 3900 3050
+$Comp
+L R R5
+U 1 1 55853CF7
+P 3900 3300
+F 0 "R5" V 3980 3300 40  0000 C CNN
+F 1 "1K" V 3907 3301 40  0000 C CNN
+F 2 "~" V 3830 3300 30  0000 C CNN
+F 3 "~" H 3900 3300 30  0000 C CNN
+	1    3900 3300
+	1    0    0    -1
+$EndComp
+Wire Wire Line
+	3900 3550 3900 3800
+Connection ~ 3900 3800
+Wire Wire Line
+	3900 2700 4750 2700
 $EndSCHEMATC
